File: PCB/REV_A/HelmetHUD/MainBoardSchematic.sch (EAGLE design)
At the start: 9 parts, among them U1 AD9389BBSTZ-165, U3 Value

Commit message: Schematic V1
Parts:
- added U$3: HDMI_A, HelmetHUD:HDMI_A
- U$2: device adafruit:MICROSD -> HelmetHUD:MICROSD
Connections:
- new net EPIOS0: U2.A0, U2.DQ0, U3A.PH0
- new net EPIOS1: U2.A1, U2.DQ1, U3A.PH1
- new net EPIOS10: U2.A10, U2.DQ10, U3A.PG1
- new net EPIOS11: U2.A11, U2.DQ11, U3A.PG0
- new net EPIOS12: U2.A12, U2.DQ12, U3B.PM3
- new net EPIOS13: U2.BA0, U2.DQ13, U3B.PM2
- new net EPIOS14: U2.BA1, U2.DQ14, U3B.PM1
- new net EPIOS15: U2.DQ15, U3B.PM0
- new net EPIOS16: U2.DQML, U3B.PL0
- new net EPIOS17: U2.DQMH, U3B.PL1
- new net EPIOS18: U2.CAS, U3B.PL2
- new net EPIOS19: U2.RAS, U3B.PL3
- new net EPIOS2: U2.A2, U2.DQ2, U3A.PH2
- new net EPIOS28: U2.WE, U3A.PB3
- new net EPIOS29: U2.CS, U3B.PN2
- new net EPIOS3: U2.A3, U2.DQ3, U3A.PH3
- new net EPIOS30: U2.CKE, U3B.PN3
- new net EPIOS31: U2.CLK, U3A.PK5
- new net EPIOS4: U2.A4, U2.DQ4, U3A.PC7
- new net EPIOS5: U2.A5, U2.DQ5, U3A.PC6
- new net EPIOS6: U2.A6, U2.DQ6, U3A.PC5
- new net EPIOS7: U2.A7, U2.DQ7, U3A.PC4
- new net EPIOS8: U2.DQ8, U3A.PA6
- new net EPIOS9: U2.DQ9, U3A.PA7
- new net GPIOA0: U3A.PA0
- new net GPIOA1: U3A.PA1
- new net GPIOA2: U3A.PA2
- new net GPIOA3: U3A.PA3
- new net GPIOC0: U3A.PC0_TCK_SWCLK
- new net GPIOC1: U3A.PC1_TMS_SWDIO
- new net GPIOC2: U3A.PC2_TDI
- new net GPIOC3: U3A.PC3_TDO_SWO
- new net GPIOD0: U3A.PD0
- new net GPIOD1: U3A.PD1
- new net GPIOD2: U3A.PD2
- new net GPIOD3: U3A.PD3
- new net GPIOD4: U3A.PD4
- new net GPIOD5: U3A.PD5
- new net GPIOD6: U3A.PD6
- new net GPIOD7: U3A.PD7
- new net GPIOK0: U3A.PK0
- new net GPIOK1: U3A.PK1
- new net GPIOK2: U3A.PK2
- new net GPIOK3: U3A.PK3
- new net GPIOL4: U3B.PL4
- new net GPIOL5: U3B.PL5
- new net GPIOL6: U3B.PL6
- new net GPIOL7: U3B.PL7
Other:
- moved on the sheet: U$1, U1, U2, U3A, U3B, U3C, U3D, X2-1, X2-2, X3-1, X3-2, X4-1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

Commit message: Schematic V2
Parts:
- added C1, C2, C3, C4, C5, C6, C7, C8, C9: (no value), SparkFun-Capacitors:0.1UF-50V-20%(PTH)KIT-EZ
- added R1: 10K, SparkFun-Passives:RESISTOR1206
- added R2: 887, SparkFun-Passives:RESISTOR1206
- added R3: 2.2K, SparkFun-Passives:RESISTOR1206
- added R4, R5: 2K, SparkFun-Passives:RESISTOR1206
- added X1: 1365-10, HelmetHUD:1365-10
Connections:
- removed net GPIOC0: U3A.PC0_TCK_SWCLK
- removed net GPIOC1: U3A.PC1_TMS_SWDIO
- removed net GPIOC2: U3A.PC2_TDI
- removed net GPIOC3: U3A.PC3_TDO_SWO
- new net 1.8V: C1.2, C2.2, C3.2, C4.2, C5.2, C6.2, C7.2, U1.1, U1.16, U1.19, U1.20, U1.21, U1.24, U1.29, U1.36, U1.41, U1.61, U1.62, U1.63, U1.64
- new net 3.3V: U$1.VDD, U$2.VDD, U2.VDD1, U2.VDD2, U2.VDD3, U2.VDDQ1, U2.VDDQ2, U2.VDDQ3, U2.VDDQ4, U3D.VDD, U3D.VDDA, U3D.VDD_10, U3D.VDD_11, U3D.VDD_12, U3D.VDD_13, U3D.VDD_14, U3D.VDD_2, U3D.VDD_3, U3D.VDD_4, U3D.VDD_5, U3D.VDD_6, U3D.VDD_7, U3D.VDD_8, U3D.VDD_9, U3D.VREFA+, X1-1.S
- new net 5V: R4.1, R5.1, U$3.VCC
- new net DDCSCL: R5.2, U$3.SCL, U1.44
- new net DDCSDA: R4.2, U$3.SDA, U1.45
- new net GND: C1.1, C2.1, C3.1, C4.1, C5.1, C6.1, C7.1, C9.2, R1.1, R2.1, U$1.AGND, U$1.GND, U$1.GND1, U$1.GND2, U$1.GND3, U$1.GND4, U$1.GND5, U$1.GND6, U$1.GND7, U$1.GND8, U$1.GND9, U$2.GND, U$2.GND1, U$2.VSS, U$3.P$17, U1.15, U1.17, U1.18, U1.22, U1.26, U1.32, U1.39, U1.42, U1.43, U1.59, U1.60, U1.79, U1.80, U2.VSS1, U2.VSS2, U2.VSS3, U2.VSSQ1, U2.VSSQ2, U2.VSSQ3, U2.VSSQ4, U3D.GND, U3D.GNDA, U3D.GND_2, U3D.GND_3, U3D.GND_4, U3D.GND_5, U3D.GND_6, X1-3.S, X1-5.S, X1-9.S
- new net GPIOE0: U$1.GPIO4, U3A.PE0
- new net GPIOE1: U$1.GPIO7, U3A.PE1
- new net GPIOE2: U$1.GPIO9, U3A.PE2
- new net GPIOM4: U1.57, U3B.PM4
- new net GPIOM5: U1.56, U3B.PM5
- new net GPIOM6: U1.55, U3B.PM6
- new net GPIOM7: U1.54, U3B.PM7
- new net HDMI_DE: U1.3, U3B.PN1
- new net HDMI_INT: U1.40, U3B.PN5
- new net N$1: R1.2, U$3.HPD, U1.25
- new net N$10: U$3.TXC+, U1.28
- new net N$11: U$3.TXC-, U1.27
- new net N$12: R3.1, U$1.MIC_BIAS
- new net N$13: C8.2, R3.2, X4-2.S
- new net N$14: U$1.MIC_R-, X4-1.S
- new net N$15: U$1.SPKR_L+, X2-1.S
- new net N$16: U$1.SPKR_R+, X2-2.S
- new net N$17: U$1.SPKR_L-, X3-1.S
- new net N$18: U$1.SPKR_R-, X3-2.S
- new net N$19: U$1.PWREN
- new net N$2: R2.2, U1.23
- new net N$20: U$2.DATA_IN, U3A.PJ1
- new net N$21: U$2.SCLK
- new net N$22: U$2.CS, U3A.PJ0
- new net N$23: C9.1, U3D.VDDC, U3D.VDDC_2
- new net N$24: U3C.RST_N, X1-10.S
- new net N$3: U$3.TX1-, U1.34
- new net N$4: U$3.TX0-, U1.30
- new net N$5: U$3.TX0+, U1.31
- new net N$6: U$3.TX1+, U1.35
- new net N$7: U$3.TX2-, U1.37
- new net N$8: C8.1, U$1.MIC_R+
- new net N$9: U$3.TX2+, U1.38
- new net SWCLK: U3A.PC0_TCK_SWCLK, X1-4.S
- new net TDI: U3A.PC2_TDI, X1-8.S
- new net TDO_SWO: U3A.PC3_TDO_SWO, X1-6.S
- new net TMS_SWDIO: U3A.PC1_TMS_SWDIO, X1-2.S
- new net U3CTS: U$1.UART_CTS
- new net U3RTS: U$1.UART_RTS, U3B.PN4
- new net U3RX: U$1.UART_TX, U3A.PA4
- new net U3TX: U$1.UART_RX, U3A.PA5
- net EPIOS8: now also U2.A9
- net EPIOS9: now also U2.A8
- net GPIOA0: now also U1.67
- net GPIOA1: now also U1.66
- net GPIOA2: now also U1.65
- net GPIOA3: now also U1.58
- net GPIOD0: now also U1.2
- net GPIOD1: now also U1.78
- net GPIOD2: now also U1.77
- net GPIOD3: now also U1.76
- net GPIOD4: now also U1.75
- net GPIOD5: now also U1.74
- net GPIOD6: now also U1.73
- net GPIOD7: now also U1.72
- net GPIOK0: now also U1.71
- net GPIOK1: now also U1.70
- net GPIOK2: now also U1.69
- net GPIOK3: now also U1.68
- net GPIOL4: now also U1.53
- net GPIOL5: now also U1.52
- net GPIOL6: now also U1.51
- net GPIOL7: now also U1.50
Other:
- moved on the sheet: U$1, U$3, U1, U2, U3A, U3B, U3C, U3D, X2-1, X2-2, X3-1, X3-2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

Commit message: Schematic V3
Parts:
- added C10, C11: (no value), SparkFun-Capacitors:0.1UF-50V-20%(PTH)KIT-EZ
Connections:
- net EPIOS10 renamed SDRAM_10
- net EPIOS11 renamed SDRAM_11
- net EPIOS12 renamed SDRAM_12
- net EPIOS13 renamed SDRAM_13
- net EPIOS14 renamed SDRAM_14
- net EPIOS15 renamed SDRAM_15
- net EPIOS16 renamed SDRAM_LDQM
- net EPIOS17 renamed SDRAM_UDQM
- net EPIOS18 renamed SDRAM_CAS
- net EPIOS19 renamed SDRAM_RAS
- net EPIOS28 renamed SDRAM_WE
- net EPIOS31 renamed SDRAM_CLK
- net EPIOS4 renamed SDRAM_4
- net EPIOS5 renamed SDRAM_5
- net EPIOS6 renamed SDRAM_6
- net EPIOS7 renamed SDRAM_7
- removed net EPIOS0: U2.A0, U2.DQ0, U3A.PH0
- removed net EPIOS1: U2.A1, U2.DQ1, U3A.PH1
- removed net EPIOS2: U2.A2, U2.DQ2, U3A.PH2
- removed net EPIOS29: U2.CS, U3B.PN2
- removed net EPIOS3: U2.A3, U2.DQ3, U3A.PH3
- removed net EPIOS30: U2.CKE, U3B.PN3
- removed net EPIOS8: U2.A9, U2.DQ8, U3A.PA6
- removed net EPIOS9: U2.A8, U2.DQ9, U3A.PA7
- removed net GPIOA0: U1.67, U3A.PA0
- removed net GPIOA1: U1.66, U3A.PA1
- removed net GPIOA2: U1.65, U3A.PA2
- removed net GPIOA3: U1.58, U3A.PA3
- removed net GPIOD0: U1.2, U3A.PD0
- removed net GPIOD1: U1.78, U3A.PD1
- removed net GPIOD2: U1.77, U3A.PD2
- removed net GPIOD3: U1.76, U3A.PD3
- removed net GPIOD4: U1.75, U3A.PD4
- removed net GPIOD5: U1.74, U3A.PD5
- removed net GPIOD6: U1.73, U3A.PD6
- removed net GPIOD7: U1.72, U3A.PD7
- removed net GPIOE0: U$1.GPIO4, U3A.PE0
- removed net GPIOE1: U$1.GPIO7, U3A.PE1
- removed net GPIOE2: U$1.GPIO9, U3A.PE2
- removed net GPIOK0: U1.71, U3A.PK0
- removed net GPIOK1: U1.70, U3A.PK1
- removed net GPIOK2: U1.69, U3A.PK2
- removed net GPIOK3: U1.68, U3A.PK3
- removed net GPIOL4: U1.53, U3B.PL4
- removed net GPIOL5: U1.52, U3B.PL5
- removed net GPIOL6: U1.51, U3B.PL6
- removed net GPIOL7: U1.50, U3B.PL7
- removed net GPIOM4: U1.57, U3B.PM4
- removed net GPIOM5: U1.56, U3B.PM5
- removed net GPIOM6: U1.55, U3B.PM6
- removed net GPIOM7: U1.54, U3B.PM7
- removed net N$14: U$1.MIC_R-, X4-1.S
- removed net N$20 (its old number): U$2.DATA_IN, U3A.PJ1
- removed net N$21: U$2.SCLK
- removed net N$22: U$2.CS, U3A.PJ0
- removed net U3CTS: U$1.UART_CTS
- removed net U3RTS: U$1.UART_RTS, U3B.PN4
- removed net U3RX: U$1.UART_TX, U3A.PA4
- removed net U3TX: U$1.UART_RX, U3A.PA5
- new net BT_GPIO7: U$1.GPIO7, U3A.PH2
- new net BT_GPIO9: U$1.GPIO9, U3A.PH3
- new net BT_UART_CTS: U$1.UART_CTS, U3A.PH1
- new net BT_UART_RTS: U$1.UART_RTS, U3A.PH0
- new net BT_UART_RX: U$1.UART_RX, U3A.PA1
- new net BT_UART_TX: U$1.UART_TX, U3A.PA0
- new net HDMI_CLK: U3A.PD1
- new net HDMI_D0: U1.2, U3A.PD6
- new net HDMI_D1: U1.78, U3B.PN1
- new net HDMI_D10: U1.69, U3A.PB4
- new net HDMI_D11: U1.68, U3A.PE4
- new net HDMI_D12: U1.67, U3A.PE5
- new net HDMI_D13: U1.66, U3A.PD4
- new net HDMI_D14: U1.65, U3A.PD5
- new net HDMI_D15: U1.58, U3A.PD2
- new net HDMI_D16: U1.57, U3A.PD3
- new net HDMI_D17: U1.56, U3B.PQ0
- new net HDMI_D18: U1.55, U3B.PQ1
- new net HDMI_D19: U1.54, U3B.PQ2
- new net HDMI_D2: U1.77, U3B.PN2
- new net HDMI_D20: U1.53, U3A.PE3
- new net HDMI_D21: U1.52, U3A.PE2
- new net HDMI_D22: U1.51, U3A.PE1
- new net HDMI_D23: U1.50, U3A.PE0
- new net HDMI_D3: U1.76, U3B.PN3
- new net HDMI_D4: U1.75, U3B.PN4
- new net HDMI_D5: U1.74, U3B.PN5
- new net HDMI_D6: U1.73, U3A.PJ0
- new net HDMI_D7: U1.72, U3B.PP0
- new net HDMI_D8: U1.71, U3B.PP1
- new net HDMI_D9: U1.70, U3A.PB5
- new net HDMI_HSYNC: U3A.PD7
- new net HDMI_VSYNC: U3A.PD0
- new net N$11: C10.2, U$1.MIC_R-
- new net SDRAM_0: U2.A0, U2.DQ0, U3A.PK0
- new net SDRAM_1: U2.A1, U2.DQ1, U3A.PK1
- new net SDRAM_2: U2.A2, U2.DQ2, U3A.PK2
- new net SDRAM_3: U2.A3, U2.DQ3, U3A.PK3
- new net SDRAM_8: U2.A8, U2.DQ8, U3A.PA6
- new net SDRAM_9: U2.A9, U2.DQ9, U3A.PA7
- new net SDRAM_CKE: U2.CKE, U3B.PP3
- new net SDRAM_CS: U2.CS, U3B.PP2
- new net SD_CS: U$2.CS, U3A.PB1
- new net SD_DIN: U$2.DATA_IN, U3A.PB2
- new net SD_SCLK: U$2.SCLK, U3A.PB0
- net GND: now also C11.1, U$3.TX0SHLD, U$3.TX1SHLD, U$3.TX2SHLD, U$3.TXCSHLD, X4-2.S
- net HDMI_DE: now also U3B.PN0; no longer U3B.PN1
- net HDMI_INT: now also U3B.PP5; no longer U3B.PN5
- net N$12: now also C11.2, C8.1
- net N$13: now also C10.1, X4-1.S; no longer C8.2, X4-2.S
- net N$8: now also C8.2; no longer C8.1
Other:
- moved on the sheet: C1, C5, C6, C7, C8, R3, X4-1, X4-2

Commit message: Schematic V4
Parts:
- added C12: 0.1 uF, SparkFun-Passives:CAP0603-CAP
- added C13: 1 uF, SparkFun-Passives:CAP0603-CAP
- added C14, C16, C19, C20, C21, C22, C23, C24, C25, C26, C28: 0.1uF, SparkFun-Passives:CAP0603-CAP
- added C15, C31, C32, C33, C34, C35, C36: 2.2 uF, SparkFun-Passives:CAP0603-CAP
- added C17, C18, C27: 0.01uF, SparkFun-Passives:CAP0603-CAP
- added C29: 10nF, SparkFun-Passives:CAP_POL6032
- added C30, C37, C44, C45: 4.7uF, SparkFun-Passives:CAP0603-CAP
- added C38, C39: 12pF, SparkFun-Passives:CAP0603-CAP
- added C40, C41: .1uF, SparkFun-Passives:CAP0603-CAP
- added C42: 4.7pF, SparkFun-Passives:CAP0603-CAP
- added C43: 22uF, SparkFun-Passives:CAP0603-CAP
- added C46: 2.2uF, SparkFun-Passives:CAP0603-CAP
- added C47: 10uF, SparkFun-Passives:CAP0603-CAP
- added C48: 1uF, SparkFun-Passives:CAP0603-CAP
- added C49: 220nF, SparkFun-Passives:CAP0603-CAP
- added D1: RED, HelmetHUD:LED-RED0603
- added D2: 1N5817-T, diode:1N5817-T
- added L1, L3: 10uH, SparkFun-Passives:INDUCTOR0603
- added L2: 4.7uH, SparkFun-Passives:INDUCTOR0603
- added R10: 750, SparkFun-Passives:RESISTOR0603-RES
- added R11: 2k, SparkFun-Passives:RESISTOR0603-RES
- added R12, R7, R8, R9: 10k, SparkFun-Passives:RESISTOR0603-RES
- added R13, R14, R23: 8, SparkFun-Passives:RESISTOR1206
- added R15: 1M, SparkFun-Passives:RESISTOR0603-RES
- added R16: 30k, SparkFun-Passives:RESISTOR0603-RES
- added R17: 82k, SparkFun-Passives:RESISTOR0603-RES
- added R18: 549k, SparkFun-Passives:RESISTOR0603-RES
- added R19: 1.65M, SparkFun-Passives:RESISTOR0603-RES
- added R20: 1k, SparkFun-Passives:RESISTOR0603-RES
- added R21: 200k, SparkFun-Passives:RESISTOR0603-RES
- added R22: 33m, SparkFun-Passives:RESISTOR0603-RES
- added R6: 470, SparkFun-Passives:RESISTOR0603-RES
- added S1: (no value), SparkFun-Retired:TAC_SWITCHPTH
- added U$4: LTC3531, HelmetHUD:LTC3531
- added U$5: LTC3405A, HelmetHUD:LTC3405A
- added U$6: LTC3401, HelmetHUD:LTC3401
- added U$7: STC3100, HelmetHUD:STC3100
- added U5: MCP73831, SparkFun-PowerIC:MCP73831
- added X5: 87438-04, con-molex:87438-04
- added X6: 87758-2016, HelmetHUD:87758-2016
- added Y1: (no value), HelmetHUD:CRYSTAL
- C1, C2, C3, C5, C6: value (none) -> .1uF; device SparkFun-Capacitors:0.1UF-50V-20%(PTH)KIT-EZ -> SparkFun-Passives:CAP0603-CAP
- C4: value (none) -> 4.7uF; device SparkFun-Capacitors:0.1UF-50V-20%(PTH)KIT-EZ -> SparkFun-Passives:CAP0603-CAP
- C7: value (none) -> 470pF; device SparkFun-Capacitors:0.1UF-50V-20%(PTH)KIT-EZ -> SparkFun-Passives:CAP0603-CAP
- C9: value (none) -> 0.01 uF; device SparkFun-Capacitors:0.1UF-50V-20%(PTH)KIT-EZ -> SparkFun-Passives:CAP0603-CAP
- R1: value 10K -> 887; device SparkFun-Passives:RESISTOR1206 -> SparkFun-Passives:RESISTOR0603-RES
- R2: value 887 -> 8
- R4: value 2K -> 2k; device SparkFun-Passives:RESISTOR1206 -> SparkFun-Passives:RESISTOR0603-RES
- R5: value 2K -> 8
Connections:
- removed net SD_SCLK: U$2.SCLK, U3A.PB0
- new net CAM_CLK: U3A.PF1, X6-1.S
- new net CAM_D0: U3B.PM5, X6-13.S
- new net CAM_D1: U3B.PM6, X6-15.S
- new net CAM_D2: U3B.PM7, X6-17.S
- new net CAM_D3: U3A.PF2, X6-19.S
- new net CAM_D4: U3A.PF3, X6-20.S
- new net CAM_D5: U3A.PF4, X6-18.S
- new net CAM_D6: U3A.PA2, X6-16.S
- new net CAM_D7: U3A.PA3, X6-14.S
- new net CAM_HSYNC: U3B.PL4, X6-9.S
- new net CAM_PCLK: U3B.PM4, X6-11.S
- new net CAM_PWDWN: U3B.PQ3, X6-12.S
- new net CAM_SCL: U3A.PB0, X6-3.S
- new net CAM_SDA: U3A.PB1, X6-5.S
- new net CAM_VSYNC: U3B.PL5, X6-7.S
- new net GAUGE_SCL: U$7.SCL, U3A.PK6
- new net GAUGE_SDA: U$7.SDA, U3A.PK7
- new net N$14: R6.2, S1.1, S1.2
- new net N$21: C30.1, R9.1, U4.VBUS, U5.VIN
- new net N$22: C37.1, C4.1, C44.1, C46.1, L1.1, R15.2, U$4.SHDN_N, U$4.VIN, U$5.RUN, U$5.VIN, U$6.VIN, U5.VBAT, X5-1.S
- new net N$25: C38.1, R10.1, Y1.1
- new net N$26: U5.PROG
- new net N$27: C39.1, U3C.OSC0, Y1.2
- new net N$28: R8.2
- new net N$29: R10.2, U3C.OSC1
- new net N$30: R14.1, X3-2.S
- new net N$31: R2.1, X3-1.S
- new net N$32: R5.1, X2-2.S
- new net N$33: R13.1, X2-1.S
- new net N$34: D1.A, R9.2
- new net N$35: D1.C, U5.STAT
- new net N$36: R15.1, U$6.SHDN_N
- new net N$37: R16.2, U$6.RT
- new net N$38: C42.1, C7.1, U$6.VC
- new net N$39: C7.2, R17.2
- new net N$40: R18.2, R19.2, U$6.FB
- new net N$41: C43.1, D2.C, R19.1, U$6.VOUT
- new net N$42: D2.A, L1.2, U$6.SW
- new net N$43: C45.1, L2.1, U$5.VOUT
- new net N$44: L2.2, U$5.SW
- new net N$45: L3.2, U$4.SW1
- new net N$46: L3.1, U$4.SW2
- new net N$47: C47.1, U$4.VOUT
- new net N$48: C48.1, R20.2, U$7.VCC
- new net N$49: C49.2, R20.1, U$7.VIN
- new net N$50: R21.2, U$7.ROSC
- new net N$51: R22.2, U$7.CG, X5-2.S
- new net N$52: U$2.SCLK, U3A.PK4
- new net N$65: X6-8.S
- new net N$66: X6-10.S
- new net SD_IN: U3A.PA4
- net 1.8V: now also C40.2, C41.2; no longer C4.2, C7.2
- net 3.3V: now also C14.1, C16.1, C17.1, C18.1, C19.1, C20.1, C21.1, C22.1, C23.1, C24.1, C25.1, C26.1, C27.1, C28.1, C31.1, C32.1, C33.1, C34.1, C35.1, C36.1, R23.1, R7.2, U$1.PWREN, U3D.VBAT, X6-2.S
- net 5V: now also R11.2, R4.2; no longer R4.1, R5.1
- net DDCSCL: now also R4.1; no longer R5.2
- net DDCSDA: now also R11.1; no longer R4.2
- net GND: now also C12.1, C13.1, C14.2, C15.1, C16.2, C17.2, C18.2, C19.2, C20.2, C21.2, C22.2, C23.2, C24.2, C25.2, C26.2, C27.2, C28.2, C29.-, C30.2, C31.2, C32.2, C33.2, C34.2, C35.2, C36.2, C37.2, C38.2, C39.2, C4.2, C40.1, C41.1, C42.2, C43.2, C44.2, C45.2, C46.2, C47.2, C48.2, C49.1, C9.1, R1.2, R12.2, R16.1, R17.1, R18.1, R21.1, R22.1, R8.1, S1.3, S1.4, U$4.GND, U$5.GND, U$5.MODE, U$6.GND, U$7.GND, U1.10, U1.11, U1.12, U1.13, U1.14, U1.7, U1.8, U1.9, U4.GND, U5.VSS, X6-6.S; no longer C4.1, C7.1, C9.2, R1.1, R2.1
- net HDMI_CLK: now also U1.6, U3A.PF0; no longer U3A.PD1
- net N$1: now also R12.1; no longer R1.2
- net N$15: now also R13.2; no longer X2-1.S
- net N$16: now also R5.2; no longer X2-2.S
- net N$17: now also R2.2; no longer X3-1.S
- net N$18: now also R14.2; no longer X3-2.S
- net N$19: now also R23.2, X6-4.S; no longer U$1.PWREN
- net N$2: now also R1.1; no longer R2.2
- net N$23: now also C12.2, C13.2, C15.2, C9.2; no longer C9.1
- net N$24: now also C29.+, R6.1, R7.1; no longer X1-10.S
- net SD_CS: now also U3A.PA5; no longer U3A.PB1
- net SD_DIN: no longer U3A.PB2
Other:
- moved on the sheet: C1, C10, C11, C2, C3, C4, C5, C6, C7, C8, C9, R1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
