File: PCB/REV_A/HelmetHUD/MainBoardSchematic.brd (EAGLE design)
At the start: 100 x 80 mm, 27 parts, among them U1 AD9389BBSTZ-165, U3 Value, X1 1365-10

Commit message: Schematic V4
Parts:
- added C12: 0.1 uF, SparkFun-Passives:0603-CAP
- added C13: 1 uF, SparkFun-Passives:0603-CAP
- added C14, C16, C19, C20, C21, C22, C23, C24, C25, C26, C28: 0.1uF, SparkFun-Passives:0603-CAP
- added C15, C31, C32, C33, C34, C35, C36: 2.2 uF, SparkFun-Passives:0603-CAP
- added C17, C18, C27: 0.01uF, SparkFun-Passives:0603-CAP
- added C29: 10nF, SparkFun-Passives:EIA6032
- added C30, C37, C44, C45: 4.7uF, SparkFun-Passives:0603-CAP
- added C38, C39: 12pF, SparkFun-Passives:0603-CAP
- added C40, C41: .1uF, SparkFun-Passives:0603-CAP
- added C42: 4.7pF, SparkFun-Passives:0603-CAP
- added C43: 22uF, SparkFun-Passives:0603-CAP
- added C46: 2.2uF, SparkFun-Passives:0603-CAP
- added C47: 10uF, SparkFun-Passives:0603-CAP
- added C48: 1uF, SparkFun-Passives:0603-CAP
- added C49: 220nF, SparkFun-Passives:0603-CAP
- added D1: RED, HelmetHUD:LED-0603
- added D2: 1N5817-T, diode:DO41-7.6
- added L1, L3: 10uH, SparkFun-Passives:0603
- added L2: 4.7uH, SparkFun-Passives:0603
- added R10: 750, SparkFun-Passives:0603-RES
- added R11: 2k, SparkFun-Passives:0603-RES
- added R12, R7, R8, R9: 10k, SparkFun-Passives:0603-RES
- added R13, R14, R23: 8, SparkFun-Passives:1206
- added R15: 1M, SparkFun-Passives:0603-RES
- added R16: 30k, SparkFun-Passives:0603-RES
- added R17: 82k, SparkFun-Passives:0603-RES
- added R18: 549k, SparkFun-Passives:0603-RES
- added R19: 1.65M, SparkFun-Passives:0603-RES
- added R20: 1k, SparkFun-Passives:0603-RES
- added R21: 200k, SparkFun-Passives:0603-RES
- added R22: 33m, SparkFun-Passives:0603-RES
- added R6: 470, SparkFun-Passives:0603-RES
- added S1: (no value), SparkFun-Retired:TACTILE-PTH
- added U$4: LTC3531, HelmetHUD:SOT23-6
- added U$5: LTC3405A, HelmetHUD:SOT23-6
- added U$6: LTC3401, HelmetHUD:MSOP10
- added U$7: STC3100, HelmetHUD:MSOP8
- added U5: MCP73831, SparkFun-PowerIC:SOT23-5
- added X5: 87438-04, con-molex:87438-04
- added X6: 87758-2016, HelmetHUD:87758-2016
- added Y1: (no value), HelmetHUD:NX5032GA
- C1, C2, C3, C5, C6: value (none) -> .1uF; device SparkFun-Capacitors:CAP-PTH-SMALL-KIT -> SparkFun-Passives:0603-CAP
- C4: value (none) -> 4.7uF; device SparkFun-Capacitors:CAP-PTH-SMALL-KIT -> SparkFun-Passives:0603-CAP
- C7: value (none) -> 470pF; device SparkFun-Capacitors:CAP-PTH-SMALL-KIT -> SparkFun-Passives:0603-CAP
- C9: value (none) -> 0.01 uF; device SparkFun-Capacitors:CAP-PTH-SMALL-KIT -> SparkFun-Passives:0603-CAP
- R1: value 10K -> 887; device SparkFun-Passives:1206 -> SparkFun-Passives:0603-RES
- R2: value 887 -> 8
- R4: value 2K -> 2k; device SparkFun-Passives:1206 -> SparkFun-Passives:0603-RES
- R5: value 2K -> 8
- moved C2 151.1 mm to (89.9, 61.6), flipped to the bottom, turned to 270 degrees
- moved C1 150.4 mm to (95.5, 61.6), flipped to the bottom, turned to 270 degrees
- moved C3 149.8 mm to (82.3, 61.6), flipped to the bottom, turned to 270 degrees
- moved C9 129.8 mm to (76.4, 42.7), flipped to the bottom
- moved C10 122.9 mm to (54.7, 12.5)
- moved C11 122.9 mm to (54.7, 8.65)
- moved C6 122.9 mm to (92.5, 61.6), flipped to the bottom, turned to 270 degrees
- moved X4 118.1 mm to (39.2, 4.96)
- moved R4 114.8 mm to (71.3, 61.6), flipped to the bottom, turned to 270 degrees
- moved C8 114.3 mm to (54.1, 16.7)
- moved C5 109.1 mm to (84.8, 61.6), flipped to the bottom, turned to 270 degrees
- moved R1 105.2 mm to (76.9, 61.6), flipped to the bottom, turned to 270 degrees
- moved U4 102.5 mm to (50.0, 2.71), turned to 90 degrees
- moved R3 102.1 mm to (45.9, 11.8)
- moved R5 100.5 mm to (33.8, 11.8)
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Connections:
- removed net SD_SCLK: U$2.5, U3.95
- removed net VBAT: U3.68
- new net CAM_CLK: U3.43, X6.1
- new net CAM_D0: U3.73, X6.13
- new net CAM_D1: U3.72, X6.15
- new net CAM_D2: U3.71, X6.17
- new net CAM_D3: U3.44, X6.19
- new net CAM_D4: U3.45, X6.20
- new net CAM_D5: U3.46, X6.18
- new net CAM_D6: U3.35, X6.16
- new net CAM_D7: U3.36, X6.14
- new net CAM_HSYNC: U3.85, X6.9
- new net CAM_PCLK: U3.74, X6.11
- new net CAM_PWDWN: U3.27, X6.12
- new net CAM_SCL: U3.95, X6.3
- new net CAM_SDA: U3.96, X6.5
- new net CAM_VSYNC: U3.86, X6.7
- new net GAUGE_SCL: U$7.4, U3.61
- new net GAUGE_SDA: U$7.3, U3.60
- new net N$14: R6.2, S1.1, S1.2
- new net N$21: C30.1, R9.1, U4.VBUS, U5.4
- new net N$22: C37.1, C4.1, C44.1, C46.1, L1.1, R15.2, U$4.4, U$4.5, U$5.1, U$5.4, U$6.3, U5.3, X5.1
- new net N$25: C38.1, R10.1, Y1.P$1
- new net N$26: U5.5
- new net N$27: C39.1, U3.88, Y1.P$2
- new net N$28: R8.2
- new net N$29: R10.2, U3.89
- new net N$30: R14.1, X3.2
- new net N$31: R2.1, X3.1
- new net N$32: R5.1, X2.2
- new net N$33: R13.1, X2.1
- new net N$34: D1.A, R9.2
- new net N$35: D1.C, U5.1
- new net N$36: R15.1, U$6.10
- new net N$37: R16.2, U$6.1
- new net N$38: C42.1, C7.1, U$6.9
- new net N$39: C7.2, R17.2
- new net N$40: R18.2, R19.2, U$6.8
- new net N$41: C43.1, D2.C, R19.1, U$6.7
- new net N$42: D2.A, L1.2, U$6.4
- new net N$43: C45.1, L2.1, U$5.5
- new net N$44: L2.2, U$5.3
- new net N$45: L3.2, U$4.6
- new net N$46: L3.1, U$4.1
- new net N$47: C47.1, U$4.3
- new net N$48: C48.1, R20.2, U$7.7
- new net N$49: C49.2, R20.1, U$7.8
- new net N$50: R21.2, U$7.2
- new net N$51: R22.2, U$7.6, X5.2
- new net N$52: U$2.5, U3.63
- new net N$65: X6.8
- new net N$66: X6.10
- new net SD_IN: U3.37
- net 1.8V: now also C40.2, C41.2; no longer C4.2, C7.2
- net 3.3V: now also C14.1, C16.1, C17.1, C18.1, C19.1, C20.1, C21.1, C22.1, C23.1, C24.1, C25.1, C26.1, C27.1, C28.1, C31.1, C32.1, C33.1, C34.1, C35.1, C36.1, R23.1, R7.2, U$1.19, U3.68, X6.2
- net 5V: now also R11.2, R4.2; no longer R4.1, R5.1
- net DDCSCL: now also R4.1; no longer R5.2
- net DDCSDA: now also R11.1; no longer R4.2
- net GND: now also C12.1, C13.1, C14.2, C15.1, C16.2, C17.2, C18.2, C19.2, C20.2, C21.2, C22.2, C23.2, C24.2, C25.2, C26.2, C27.2, C28.2, C29.P$2, C30.2, C31.2, C32.2, C33.2, C34.2, C35.2, C36.2, C37.2, C38.2, C39.2, C4.2, C40.1, C41.1, C42.2, C43.2, C44.2, C45.2, C46.2, C47.2, C48.2, C49.1, C9.1, R1.2, R12.2, R16.1, R17.1, R18.1, R21.1, R22.1, R8.1, S1.3, S1.4, U$4.2, U$5.2, U$5.6, U$6.5, U$7.5, U1.10, U1.11, U1.12, U1.13, U1.14, U1.7, U1.8, U1.9, U4.GND, U5.2, X6.6; no longer C4.1, C7.1, C9.2, R1.1, R2.1
- net HDMI_CLK: now also U1.6, U3.42; no longer U3.2
- net N$1: now also R12.1; no longer R1.2
- net N$15: now also R13.2; no longer X2.1
- net N$16: now also R5.2; no longer X2.2
- net N$17: now also R2.2; no longer X3.1
- net N$18: now also R14.2; no longer X3.2
- net N$19: now also R23.2, X6.4; no longer U$1.19
- net N$2: now also R1.1; no longer R2.2
- net N$23: now also C12.2, C13.2, C15.2, C9.2; no longer C9.1
- net N$24: now also C29.P$1, R6.1, R7.1; no longer X1.10
- net SD_CS: now also U3.38; no longer U3.96
- net SD_DIN: no longer U3.91
Routing:
- net DDCSDA: track 0.00 -> 64.4 mm
- net DDCSCL: track 0.00 -> 59.7 mm
- net 5V: track 0.00 -> 50.9 mm, vias 0 -> 2
- net N$20: track 0.00 -> 41.7 mm
- net N$10: track 0.00 -> 41.6 mm
- net N$5: track 0.00 -> 41.4 mm
- net N$4: track 0.00 -> 41.3 mm
- net N$6: track 0.00 -> 41.0 mm
- net N$3: track 0.00 -> 40.8 mm
- net N$9: track 0.00 -> 40.8 mm
- net N$7: track 0.00 -> 40.6 mm
- net N$1: track 0.00 -> 40.6 mm
- net HDMI_DE: track 0.00 -> 35.5 mm
- net HDMI_D1: track 0.00 -> 26.1 mm
- net HDMI_D2: track 0.00 -> 25.2 mm
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- added copper zone on layer 16, net GND

Commit message: PCB REV B
Parts:
- moved C41 63.5 mm to (27.9, 39.3), flipped to the top, turned to 180 degrees
- moved C2 62.0 mm to (31.9, 39.7), flipped to the top
- moved C6 61.5 mm to (35.0, 39.7), flipped to the top
- moved C5 60.3 mm to (27.9, 41.9), flipped to the top, turned to 180 degrees
- moved C3 57.1 mm to (27.7, 44.6), flipped to the top, turned to 0 degrees
- moved C1 54.4 mm to (44.5, 42.6)
- moved R1 54.2 mm to (23.4, 69.9), turned to 180 degrees
- moved C40 53.9 mm to (27.7, 47.2), flipped to the top, turned to 0 degrees
- moved U2 48.5 mm to (85.6, 43.9)
- moved X1 47.3 mm to (51.8, 68.1), turned to 180 degrees
- moved R12 44.4 mm to (29.9, 64.4), turned to 90 degrees
- moved R4 41.2 mm to (30.4, 56.3), turned to 180 degrees
- moved X6 38.8 mm to (70.5, 60.4), turned to 315 degrees
- moved C39 38.0 mm to (57.3, 50.7), turned to 180 degrees
- moved R10 34.7 mm to (57.5, 47.6)
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Connections:
- removed net N$8: C8.2, U$1.33
- new net N$59: C11.2, U$1.33
- net GND: now also C8.1; no longer C11.1
- net N$12: now also C11.1, C8.2; no longer C11.2, C8.1
Routing:
- net 3.3V: track 0.00 -> 101.5 mm, vias 0 -> 3
- net GND: track 0.00 -> 89.0 mm, vias 0 -> 5
- net SDRAM_3: track 0.00 -> 87.3 mm
- net SDRAM_0: track 0.00 -> 85.4 mm, vias 0 -> 2
- net N$19: track 0.00 -> 78.7 mm, vias 0 -> 2
- net SDRAM_4: track 0.00 -> 75.4 mm, vias 0 -> 2
- net SDRAM_CS: track 0.00 -> 70.2 mm, vias 0 -> 4
- net SDRAM_6: track 0.00 -> 69.6 mm, vias 0 -> 4
- net SDRAM_WE: track 0.00 -> 60.5 mm, vias 0 -> 4
- net DDCSCL: track 59.7 -> 0.00 mm
- net SDRAM_RAS: track 0.00 -> 52.6 mm, vias 0 -> 4
- net 5V: track 50.9 -> 0.00 mm, vias 2 -> 0
- net N$52: track 0.00 -> 46.3 mm, vias 0 -> 2
- net SD_CS: track 0.00 -> 44.6 mm, vias 0 -> 2
- net SDRAM_13: track 0.00 -> 43.9 mm, vias 0 -> 2
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Other:
- board size 100 x 80 mm -> 99 x 80 mm
