File: PCB/REV_B/HelmetHUD/MainBoardSchematic.brd (EAGLE design)
At the start: 99 x 80 mm, 77 parts, among them U1 AD9389BBSTZ-165, U3 Value, U5 MCP73831, X1 1365-10, X5 87438-04, X6 87758-2016

Commit message: PCB REV B update
Parts:
- added C4, C7: 10uF, SparkFun-Passives:0603-CAP
- added C42, C43: 100 uF, SparkFun-Capacitors:EIA6032
- added C44: .1uF, SparkFun-Passives:0603-CAP
- added C45: 4.7 uF, SparkFun-Capacitors:CAP-PTH-SMALL-KIT
- added C47, C50: 1uF, SparkFun-Passives:0603-CAP
- added IC1: V_REG_LM1117SOT223, HelmetHUD:SOT223
- added IC2, IC3: 74AHC1G00DBV, 74xx-little-us:SOT23-5
- added R15: 15k, SparkFun-Passives:0603-RES
- added R17: 5M, SparkFun-Passives:0603-RES
- added R18, R19: 100k, SparkFun-Passives:0603-RES
- added S3: (no value), SparkFun-Retired:TACTILE-PTH
- added U$4: PTN04050C, HelmetHUD:PTN04050C
- added U$5: AXH003A0XZ, HelmetHUD:AXH003A0XZ
- U1: value AD9389BBSTZ-165 -> HDMI TX
- U2: value (none) -> SDRAM
- U3: value Value -> Cortex M4
- X6: value 87758-2016 -> Cortex 10
- moved X2 96.1 mm to (94.9, 74.5), turned to 270 degrees
- moved R13 86.7 mm to (94.6, 67.2)
- moved X5 75.5 mm to (19.4, 80.5), turned to 270 degrees
- moved R2 75.1 mm to (89.0, 68.4)
- moved X3 74.0 mm to (6.94, 78.1), turned to 90 degrees
- moved R14 61.6 mm to (14.8, 73.4), turned to 90 degrees
- moved R5 60.6 mm to (17.9, 70.3), turned to 90 degrees
- moved X4 32.6 mm to (6.64, 4.83), turned to 90 degrees
- moved U$7 31.2 mm to (42.0, 28.1)
- moved U5 30.1 mm to (14.3, 43.1), turned to 90 degrees
- moved C37 26.4 mm to (22.4, 39.6)
- moved R8 24.1 mm to (15.6, 39.5), turned to 180 degrees
- moved C30 23.4 mm to (11.6, 38.6), turned to 180 degrees
- moved R20 21.5 mm to (34.2, 40.0)
- moved C49 21.3 mm to (33.8, 43.2)
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Connections:
- removed net N$48: C48.1, R20.2, U$7.7
- removed net SD_DIN: U$2.3
- new net 3.7V: C42.P$1, IC2.2, IC3.4, U$4.P$4, U$5.P$2
- new net N$38: IC2.4, IC3.2
- new net N$40: C47.1, IC3.1, R18.1
- new net N$41: C47.2, R17.2, R19.2, S3.1, S3.2
- new net N$42: C37.1, C48.1, R18.2, R19.1, R20.2, U$7.7, U5.3, X5.1
- new net N$43: C50.2, IC2.1, R17.1
- new net SD_CD: U$2.CD1, U3.102
- new net VCC: IC2.5, IC3.5
- net 1.8V: now also U$5.P$5
- net 3.3V: now also C44.1, C45.2, C7.1, IC1.2, IC1.4
- net 5V: now also C4.1, C43.P$1, IC1.3, U$4.P$2
- net GND: now also C4.2, C42.P$2, C43.P$2, C44.2, C45.1, C50.1, C7.2, IC1.1, IC2.3, IC3.3, R15.1, S3.3, S3.4, U$2.CD2, U$4.P$1, U$5.P$3
- net N$22: now also R15.2, U$5.P$4; no longer C37.1, U5.3, X5.1
- net N$31: now also X2.2; no longer X3.1
- net N$32: now also X3.1; no longer X2.2
- net SD_IN: now also U$2.3
Routing:
- net GND: track 159.9 -> 409.9 mm, vias 8 -> 24
- net 3.3V: track 88.8 -> 335.4 mm, vias 4 -> 18
- net N$42: track 0.00 -> 151.8 mm, vias 0 -> 13
- net N$16: track 0.00 -> 135.7 mm, vias 0 -> 2
- net N$18: track 0.00 -> 130.2 mm, vias 0 -> 4
- net 1.8V: track 11.4 -> 132.9 mm, vias 0 -> 8
- net N$15: track 0.00 -> 99.9 mm, vias 0 -> 2
- net N$17: track 0.00 -> 99.1 mm, vias 0 -> 4
- net 5V: track 3.80 -> 102.5 mm, vias 0 -> 1
- net N$51: track 0.00 -> 82.0 mm, vias 0 -> 2
- net 3.7V: track 0.00 -> 69.8 mm, vias 0 -> 3
- net N$21: track 0.00 -> 66.8 mm, vias 0 -> 4
- net SD_IN: track 0.00 -> 46.0 mm, vias 0 -> 2
- net GAUGE_SDA: track 69.8 -> 35.5 mm
- net GAUGE_SCL: track 68.4 -> 38.1 mm
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Other:
- board size 99 x 80 mm -> 150 x 87.5 mm

Commit message: Add the latest PCB
Parts:
- removed C45: 4.7 uF, SparkFun-Capacitors:CAP-PTH-SMALL-KIT
- removed S3: (no value), SparkFun-Retired:TACTILE-PTH
- added C46: 4.7uF, SparkFun-Passives:0603-CAP
- added R16: 0, SparkFun-Passives:1206
- added X7: 22-23-2041, HelmetHUD:22-23-2041
- added X8: (no value), con-molex:KK-156-2
- C10, C8: value (none) -> 47 nF; device SparkFun-Capacitors:CAP-PTH-SMALL-KIT -> SparkFun-Passives:0603-CAP
- C11: value (none) -> 1uF; device SparkFun-Capacitors:CAP-PTH-SMALL-KIT -> SparkFun-Passives:0603-CAP
- IC2, IC3: value 74AHC1G00DBV -> NAND
- X1: value 1365-10 -> Cortex 10
- X6: value Cortex 10 -> Camera HDR
- moved C7 38.3 mm to (28.6, 11.2), turned to 270 degrees
- moved C4 22.8 mm to (16.1, 4.80), turned to 270 degrees
- moved C34 9.73 mm to (83.0, 56.6), flipped to the top, turned to 180 degrees
- moved C8 8.21 mm to (54.1, 12.0), turned to 0 degrees
- moved R2 5.86 mm to (94.9, 67.8), turned to 270 degrees
- moved R13 3.75 mm to (98.3, 67.8), turned to 270 degrees
- moved C10 3.44 mm to (56.4, 15.5), turned to 270 degrees
- moved C11 3.31 mm to (52.9, 17.2)
- moved C13 2.79 mm to (46.4, 42.9), turned to 45 degrees
- moved C18 0.90 mm to (82.0, 53.4)
- moved R23 0.63 mm to (63.8, 77.0)
- moved C39 0.42 mm to (61.6, 59.5)
- moved Y1 0.40 mm to (64.5, 55.7)
- moved C38 0.29 mm to (68.2, 57.0)
- moved R10 0.22 mm to (65.9, 59.2)
Connections:
- new net N$28: R16.2, U$1.36
- net 3.3V: now also C46.2; no longer C45.2
- net 3.7V: now also X7.1, X7.2
- net GND: now also C11.1, C46.1, R16.1, X7.3, X7.4, X8.1; no longer C45.1, C8.1, S3.3, S3.4, U$1.36
- net N$11: now also C8.2; no longer C10.2
- net N$12: now also C10.1, C11.2; no longer C11.1, C8.2
- net N$13: now also C8.1; no longer C10.1
- net N$41: now also X8.2; no longer S3.1, S3.2
- net N$59: now also C10.2; no longer C11.2
Routing:
- net SD_CD: track 0.03 -> 158.3 mm, vias 0 -> 2
- net GND: track 409.9 -> 513.6 mm, vias 24 -> 35
- net N$24: track 5.64 -> 100.0 mm, vias 0 -> 7
- net 3.7V: track 69.8 -> 158.6 mm
- net SDRAM_7: track 52.7 -> 105.9 mm, vias 4 -> 6
- net N$41: track 12.0 -> 50.5 mm, vias 0 -> 3
- net 5V: track 102.5 -> 136.7 mm, vias 1 -> 3
- net N$23: track 15.9 -> 32.4 mm, vias 1 -> 4
- net 3.3V: track 335.4 -> 323.6 mm, vias 18 -> 22
- net SDRAM_CS: track 61.1 -> 72.2 mm
- net N$15: track 99.9 -> 89.1 mm
- net CAM_HSYNC: track 31.7 -> 23.4 mm
- net N$16: track 135.7 -> 143.3 mm, vias 2 -> 4
- net N$33: track 17.2 -> 9.94 mm
- net N$17: track 99.1 -> 92.4 mm
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- added copper zone on layer 1, net 3.3V
Other:
- board size 150 x 87.5 mm -> 104.1 x 87.4 mm
- board text added: "3/13/2015"
- board text added: "ECE477 Group 12"
- board text added: "V1.0"
