File: PCB/REV_B/HelmetHUD/MainBoardSchematic.sch (EAGLE design)
At the start: 78 parts, among them IC1 LD117AS25TR, U1 AD9389BBSTZ-165, U3 Value, U5 MCP73831, X1 1365-10, X5 87438-04, X6 87758-2016

Commit message: PCB REV B update
Parts:
- added C4, C7: 10uF, SparkFun-Passives:CAP0603-CAP
- added C42, C43: 100 uF, SparkFun-Capacitors:CAP_POL6032
- added C44: .1uF, SparkFun-Passives:CAP0603-CAP
- added C45: 4.7 uF, SparkFun-Capacitors:0.1UF-50V-20%(PTH)KIT-EZ
- added C47, C50: 1uF, SparkFun-Passives:CAP0603-CAP
- added IC2, IC3: 74AHC1G00DBV, 74xx-little-us:74AHC1G00DBV
- added R15: 15k, SparkFun-Passives:RESISTOR0603-RES
- added R17: 5M, SparkFun-Passives:RESISTOR0603-RES
- added R18, R19: 100k, SparkFun-Passives:RESISTOR0603-RES
- added S3: (no value), SparkFun-Retired:TAC_SWITCHPTH
- added U$4: PTN04050C, HelmetHUD:PTN04050C
- added U$5: AXH003A0XZ, HelmetHUD:AXH003A0XZ
- IC1: value LD117AS25TR -> V_REG_LM1117SOT223; device v-reg:LD117AS25TR -> HelmetHUD:V_REG_LM1117SOT223
- U1: value AD9389BBSTZ-165 -> HDMI TX
- U2: value (none) -> SDRAM
- U3: value Value -> Cortex M4
- X6: value 87758-2016 -> Cortex 10
Connections:
- new net 3.7V: C42.+, IC2A.I1, IC3A.O, U$4.V_IN, U$5.V_IN
- new net N$38: IC2A.O, IC3A.I1
- new net N$40: C47.1, IC3A.I0, R18.1
- new net N$41: C47.2, R17.2, R19.2, S3.1, S3.2
- new net N$42: C37.1, C48.1, R18.2, R19.1, R20.2, U$7.VCC, U5.VBAT, X5-1.S
- new net N$43: C50.2, IC2A.I0, R17.1
- new net SD_CD: U$2.CARD_DETECT, U3B.PQ4
- net 1.8V: now also U$5.V_OUT
- net 3.3V: now also C44.1, C45.2, C7.1, IC1.OUT, IC1.OUT@1
- net 5V: now also C4.1, C43.+, IC1.IN, U$4.V_OUT
- net GND: now also C4.2, C42.-, C43.-, C44.2, C45.1, C50.1, C7.2, IC1.ADJ, R15.1, S3.3, S3.4, U$2.CARD_DETECT1, U$4.GND, U$5.GND
- net N$22: now also R15.2, U$5.TRIM; no longer C37.1, C48.1, R20.2, U$7.VCC, U5.VBAT, X5-1.S
- net N$31: now also X2-2.S; no longer X3-1.S
- net N$32: now also X3-1.S; no longer X2-2.S

Commit message: Add the latest PCB
Parts:
- removed C45: 4.7 uF, SparkFun-Capacitors:0.1UF-50V-20%(PTH)KIT-EZ
- removed S3: (no value), SparkFun-Retired:TAC_SWITCHPTH
- added C46: 4.7uF, SparkFun-Passives:CAP0603-CAP
- added R16: 0, SparkFun-Passives:RESISTOR1206
- added X7: 22-23-2041, HelmetHUD:22-23-2041
- added X8: (no value), con-molex:KK-156-2
- C10, C8: value (none) -> 47 nF; device SparkFun-Capacitors:0.1UF-50V-20%(PTH)KIT-EZ -> SparkFun-Passives:CAP0603-CAP
- C11: value (none) -> 1uF; device SparkFun-Capacitors:0.1UF-50V-20%(PTH)KIT-EZ -> SparkFun-Passives:CAP0603-CAP
- IC2, IC3: value 74AHC1G00DBV -> NAND
- X1: value 1365-10 -> Cortex 10
- X6: value Cortex 10 -> Camera HDR
Connections:
- new net N$28: R16.2, U$1.AGND
- net 3.3V: now also C46.2; no longer C45.2
- net 3.7V: now also X7-1.S, X7-2.S
- net GND: now also C11.1, C46.1, R16.1, X7-3.S, X7-4.S, X8-1.S; no longer C45.1, C8.1, S3.3, S3.4, U$1.AGND
- net N$11: now also C8.2; no longer C10.2
- net N$12: now also C10.1, C11.2; no longer C11.1, C8.2
- net N$13: now also C8.1; no longer C10.1
- net N$41: now also X8-2.S; no longer S3.1, S3.2
- net N$59: now also C10.2; no longer C11.2
Other:
- moved on the sheet: C10, C11, C8
